File: hw/opto_board.kicad_pcb (KiCad board)
At the start: 2 copper layers, 94 x 45 mm, 36 parts, among them J1 Conn_01x02, J2 DB9_Male_MountingHoles-Connec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, J4 Conn_01x03, J5 Conn_01x03, J6 Conn_01x03, J7 Conn_01x03, J8 Conn_01x03, J9 Conn_01x03, U1 MAX232N-dk_Interface-Drivers-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, U2 nucleo_nano

Commit message: updated gerber files
Connections:
- J4 pad 2: Net-(J4-Pad2) -> Net-(J4-Pad1)
- J5 pad 2: Net-(J5-Pad2) -> Net-(J5-Pad1)
- U1 pad 10: Net-(J5-Pad2) -> Net-(J5-Pad1)
- U1 pad 11: Net-(J5-Pad2) -> Net-(J5-Pad1)
- U1 pad 12: Net-(J4-Pad2) -> Net-(J4-Pad1)
Routing:
- net Net-(J4-Pad1): track 19.3 -> 33.5 mm
- net Net-(J5-Pad1): track 36.3 -> 49.2 mm
- net Net-(J4-Pad2): track 8.08 -> 0.00 mm
- net Net-(J5-Pad2): track 7.62 -> 0.00 mm
- net +3V3: track 133.2 -> 127.0 mm
Other:
- board text added: "2021-04-21"
- board text added: "RS232 to SCPI multimeter"
- board text added: "Temp"
- board text added: "current"
- board text added: "drekkar stm32 scpi"
- board text added: "fans"
- board text removed: "2021-04-06"
- board text removed: "RS-232 Opto adapter nucleo temp"
