File: hw/opto_board.sch (KiCad schematic (older format))
At the start: 36 parts, among them J1 Conn_01x02, J2 DB9_Male_MountingHoles-Connec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, J4 Conn_01x03, J5 Conn_01x03, J6 Conn_01x03, J7 Conn_01x03, J8 Conn_01x03, J9 Conn_01x03, U1 MAX232N-dk_Interface-Drivers-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, U2 nucleo_nano

Commit message: added eit_kicad_libraries
Parts:
- C1, C10, C11, C2, C3, C4, C5, C6, C7, C8, C9: symbol opto_board-rescue:C-Device -> opto_board-rescue:C-Device-opto_board-rescue
- D12, D2, D6: symbol opto_board-rescue:LED-Device -> opto_board-rescue:LED-Device-opto_board-rescue
- D4, D8: symbol opto_board-rescue:D_Zener-Device -> opto_board-rescue:D_Zener-Device-opto_board-rescue
- D7: symbol opto_board-rescue:D_Bridge_+-AA-Device -> opto_board-rescue:D_Bridge_+-AA-Device-opto_board-rescue
- J1: symbol opto_board-rescue:Conn_01x02-Connector_Generic -> opto_board-rescue:Conn_01x02-Connector_Generic-opto_board-rescue
- J4, J5, J6, J7, J8, J9: symbol opto_board-rescue:Conn_01x03-Connector_Generic -> opto_board-rescue:Conn_01x03-Connector_Generic-opto_board-rescue
- R1, R2, R3, R4, R5, R8, R9: symbol opto_board-rescue:R-Device -> opto_board-rescue:R-Device-opto_board-rescue
- U2: symbol opto_board-rescue:nucleo_nano-eit_proprietary -> opto_board-rescue:nucleo_nano-eit_proprietary-opto_board-rescue
Changed lines of the file:
@@
 $EndDescr
 $Comp
-L opto_board-rescue:LED-Device D6
+L opto_board-rescue:LED-Device-opto_board-rescue D6
 U 1 1 5E11B181
 P 4300 1800
@@
 $EndComp
 $Comp
-L opto_board-rescue:D_Zener-Device D8
+L opto_board-rescue:D_Zener-Device-opto_board-rescue D8
 U 1 1 5E171B70
 P 5200 7250
@@
 $EndComp
 $Comp
-L opto_board-rescue:GND-power-opto_board-rescue #PWR06
+L opto_board-rescue:GND-power-opto_board-rescue-opto_board-rescue #PWR06
 U 1 1 5E171B76
 P 5200 7450
@@
 $EndComp
 $Comp
-L opto_board-rescue:nucleo_nano-eit_proprietary U2
+L opto_board-rescue:nucleo_nano-eit_proprietary-opto_board-rescue U2
 U 1 1 5E112947
 P 4850 4500
@@
 $EndComp
 $Comp
-L opto_board-rescue:+5V-power-board-rescue #PWR02
+L opto_board-rescue:+5V-power-board-rescue-opto_board-rescue #PWR02
 U 1 1 5E11AF97
 P 5200 7050
@@
 $EndComp
 $Comp
-L opto_board-rescue:C-Device C4
+L opto_board-rescue:C-Device-opto_board-rescue C4
 U 1 1 5E121A04
 P 3650 2600
@@
 	1300 2100 1100 2100
 $Comp
-L opto_board-rescue:GND-power-opto_board-rescue #PWR01
+L opto_board-rescue:GND-power-opto_board-rescue-opto_board-rescue #PWR01
 U 1 1 5E1525D4
 P 1200 2900
@@
 	1200 2500 1200 2900
 $Comp
-L opto_board-rescue:GND-power-opto_board-rescue #PWR04
+L opto_board-rescue:GND-power-opto_board-rescue-opto_board-rescue #PWR04
 U 1 1 5E1A7F28
 P 2600 2550
@@
 	5550 4800 6700 4800
 $Comp
-L opto_board-rescue:GND-power-opto_board-rescue #PWR09
+L opto_board-rescue:GND-power-opto_board-rescue-opto_board-rescue #PWR09
 U 1 1 5E1B22AD
 P 6700 6650
@@
 	2600 1200 2600 1300
 $Comp
-L opto_board-rescue:+5V-power-board-rescue #PWR010
+L opto_board-rescue:+5V-power-board-rescue-opto_board-rescue #PWR010
 U 1 1 5E1D8E20
 P 7300 4400
@@
 	1300 1900 1300 2000
 $Comp
-L opto_board-rescue:Conn_01x03-Connector_Generic J5
+L opto_board-rescue:Conn_01x03-Connector_Generic-opto_board-rescue J5
 U 1 1 5E1E18D7
 P 7400 1200
@@
 	6800 5100 5550 5100
 $Comp
-L opto_board-rescue:Conn_01x03-Connector_Generic J4
+L opto_board-rescue:Conn_01x03-Connector_Generic-opto_board-rescue J4
 U 1 1 5E1EB3F0
 P 7400 800
@@
 	1400 2100 1400 2200
 $Comp
-L opto_board-rescue:R-Device R4
+L opto_board-rescue:R-Device-opto_board-rescue R4
 U 1 1 5E230F14
 P 800 1050
@@
 NoConn ~ 4150 4900
 $Comp
-L opto_board-rescue:C-Device C7
+L opto_board-rescue:C-Device-opto_board-rescue C7
 U 1 1 5E195706
 P 1600 1600
@@
 $EndComp
 $Comp
-L opto_board-rescue:C-Device C6
+L opto_board-rescue:C-Device-opto_board-rescue C6
 U 1 1 5E1958F9
 P 1600 1100
@@
 $EndComp
 $Comp
-L opto_board-rescue:C-Device C8
+L opto_board-rescue:C-Device-opto_board-rescue C8
 U 1 1 5E195975
 P 3550 1100
@@
 NoConn ~ 3200 1800
 $Comp
-L opto_board-rescue:LED-Device D12
+L opto_board-rescue:LED-Device-opto_board-rescue D12
 U 1 1 5E2292B9
 P 8600 4650
@@
 	6700 6500 3550 6500
 $Comp
-L opto_board-rescue:LED-Device D2
+L opto_board-rescue:LED-Device-opto_board-rescue D2
 U 1 1 5E3B06FE
 P 4400 7250
@@
 	4400 7400 4400 7450
 $Comp
-L opto_board-rescue:+3.3V-power-board-rescue #PWR013
+L opto_board-rescue:+3.3V-power-board-rescue-opto_board-rescue #PWR013
 U 1 1 5E126993
 P 7650 4600
@@
 	7650 4600 7650 6000
 $Comp
-L opto_board-rescue:+3.3V-power-board-rescue #PWR012
+L opto_board-rescue:+3.3V-power-board-rescue-opto_board-rescue #PWR012
 U 1 1 5E13E3D8
 P 4300 1550
@@
 $EndComp
 $Comp
-L opto_board-rescue:+3.3V-power-board-rescue #PWR014
+L opto_board-rescue:+3.3V-power-board-rescue-opto_board-rescue #PWR014
 U 1 1 5E13EBE4
 P 8600 4300
@@
 $EndComp
 $Comp
-L opto_board-rescue:+3.3V-power-board-rescue #PWR07
+L opto_board-rescue:+3.3V-power-board-rescue-opto_board-rescue #PWR07
 U 1 1 5E13F307
 P 3650 2350
@@
 	3650 2850 3650 2800
 $Comp
-L opto_board-rescue:D_Zener-Device D4
+L opto_board-rescue:D_Zener-Device-opto_board-rescue D4
 U 1 1 5E1575D8
 P 3900 2600
@@
 	3650 2800 3650 2750
 $Comp
-L opto_board-rescue:+3.3V-power-board-rescue #PWR0103
+L opto_board-rescue:+3.3V-power-board-rescue-opto_board-rescue #PWR0103
 U 1 1 5E1B6CCA
 P 2600 1200
@@
 $EndComp
 $Comp
-L opto_board-rescue:C-Device C5
+L opto_board-rescue:C-Device-opto_board-rescue C5
 U 1 1 5E1C3CE0
 P 3800 7250
@@
 $EndComp
 $Comp
-L opto_board-rescue:+3.3V-power-board-rescue #PWR0104
+L opto_board-rescue:+3.3V-power-board-rescue-opto_board-rescue #PWR0104
 U 1 1 5E1C3DCE
 P 3800 7050
@@
 $EndComp
 $Comp
-L opto_board-rescue:GND-power-opto_board-rescue #PWR0105
+L opto_board-rescue:GND-power-opto_board-rescue-opto_board-rescue #PWR0105
 U 1 1 5E1C3E79
 P 3800 7450
@@
 	3800 7050 3800 7100
 $Comp
-L opto_board-rescue:GND-power-opto_board-rescue #PWR0106
+L opto_board-rescue:GND-power-opto_board-rescue-opto_board-rescue #PWR0106
 U 1 1 5E1DC32D
 P 4400 7450
@@
 $EndComp
 $Comp
-L opto_board-rescue:+3.3V-power-board-rescue #PWR0107
+L opto_board-rescue:+3.3V-power-board-rescue-opto_board-rescue #PWR0107
 U 1 1 5E1DC4FB
 P 4400 7050
@@
 	4600 800  4600 2100
 $Comp
-L opto_board-rescue:Conn_01x03-Connector_Generic J7
+L opto_board-rescue:Conn_01x03-Connector_Generic-opto_board-rescue J7
 U 1 1 5E39CDBB
 P 1200 6400
@@
 $EndComp
 $Comp
-L opto_board-rescue:Conn_01x03-Connector_Generic J6
+L opto_board-rescue:Conn_01x03-Connector_Generic-opto_board-rescue J6
 U 1 1 5E39D0E5
 P 1200 5900
@@
 	1900 6000 4150 6000
 $Comp
-L opto_board-rescue:GND-power-opto_board-rescue #PWR0110
+L opto_board-rescue:GND-power-opto_board-rescue-opto_board-rescue #PWR0110
 U 1 1 5E3B3982
 P 1500 6700
@@
 Connection ~ 1500 6500
 $Comp
-L opto_board-rescue:+5V-power-board-rescue #PWR0111
+L opto_board-rescue:+5V-power-board-rescue-opto_board-rescue #PWR0111
 U 1 1 5E3D5CBE
 P 1600 5600
@@
 	5550 5800 8600 5800
 $Comp
-L opto_board-rescue:Conn_01x03-Connector_Generic J8
+L opto_board-rescue:Conn_01x03-Connector_Generic-opto_board-rescue J8
 U 1 1 5E45E28C
 P 10600 5300
@@
 $EndComp
 $Comp
-L opto_board-rescue:Conn_01x03-Connector_Generic J9
+L opto_board-rescue:Conn_01x03-Connector_Generic-opto_board-rescue J9
 U 1 1 5E469F67
 P 10600 5800
@@
 	9000 5500 5550 5500
 $Comp
-L opto_board-rescue:GND-power-opto_board-rescue #PWR0112
+L opto_board-rescue:GND-power-opto_board-rescue-opto_board-rescue #PWR0112
 U 1 1 5E4822FA
 P 10300 6000
@@
 Connection ~ 10300 5900
 $Comp
-L opto_board-rescue:+3.3V-power-board-rescue #PWR0113
+L opto_board-rescue:+3.3V-power-board-rescue-opto_board-rescue #PWR0113
 U 1 1 5E49B27F
 P 10200 5000
@@
 Connection ~ 10200 5300
 $Comp
-L opto_board-rescue:R-Device R8
+L opto_board-rescue:R-Device-opto_board-rescue R8
 U 1 1 5E4B522F
 P 9100 4750
@@
 $EndComp
 $Comp
-L opto_board-rescue:R-Device R9
+L opto_board-rescue:R-Device-opto_board-rescue R9
 U 1 1 5E4CEF1C
 P 9600 4750
@@
 	1900 5500 4150 5500
 $Comp
-L opto_board-rescue:GND-power-opto_board-rescue #PWR0115
+L opto_board-rescue:GND-power-opto_board-rescue-opto_board-rescue #PWR0115
 U 1 1 5E12BEB6
 P 3650 2850
@@
 $EndComp
 $Comp
-L opto_board-rescue:C-Device C9
+L opto_board-rescue:C-Device-opto_board-rescue C9
 U 1 1 5E12D248
 P 9100 6050
@@
 $EndComp
 $Comp
-L opto_board-rescue:C-Device C10
+L opto_board-rescue:C-Device-opto_board-rescue C10
 U 1 1 5E12D323
 P 9600 6000
@@
 	9600 6250 9600 6150
 $Comp
-L opto_board-rescue:GND-power-opto_board-rescue #PWR03
+L opto_board-rescue:GND-power-opto_board-rescue-opto_board-rescue #PWR03
 U 1 1 5E136410
 P 9350 6300
@@
 	9600 5850 9600 5700
 $Comp
-L opto_board-rescue:GND-power-opto_board-rescue #PWR0108
+L opto_board-rescue:GND-power-opto_board-rescue-opto_board-rescue #PWR0108
 U 1 1 5E1783A3
 P 9750 4300
@@
 	8600 4300 8600 4500
 $Comp
-L opto_board-rescue:D_Bridge_+-AA-Device D7
+L opto_board-rescue:D_Bridge_+-AA-Device-opto_board-rescue D7
 U 1 1 5E13C1AF
 P 1600 3600
@@
 	3650 4700 4150 4700
 $Comp
-L opto_board-rescue:Conn_01x02-Connector_Generic J1
+L opto_board-rescue:Conn_01x02-Connector_Generic-opto_board-rescue J1
 U 1 1 5E13D6E9
 P 800 3650
@@
 	1600 3950 1600 3900
 $Comp
-L opto_board-rescue:GND-power-opto_board-rescue #PWR0114
+L opto_board-rescue:GND-power-opto_board-rescue-opto_board-rescue #PWR0114
 U 1 1 5E154435
 P 1250 4100
@@
 	1250 3600 1250 4050
 $Comp
-L opto_board-rescue:R-Device R1
+L opto_board-rescue:R-Device-opto_board-rescue R1
 U 1 1 5E16030F
 P 2700 3800
@@
 	5900 5700 5900 3600
 $Comp
-L opto_board-rescue:C-Device C1
+L opto_board-rescue:C-Device-opto_board-rescue C1
 U 1 1 5E13D649
 P 3150 3800
@@
 NoConn ~ 5550 5300
 $Comp
-L opto_board-rescue:C-Device C11
+L opto_board-rescue:C-Device-opto_board-rescue C11
 U 1 1 5E1C3C65
 P 3900 1500
@@
 	3300 900  3300 1600
 $Comp
-L opto_board-rescue:GND-power-opto_board-rescue #PWR05
+L opto_board-rescue:GND-power-opto_board-rescue-opto_board-rescue #PWR05
 U 1 1 5E217677
 P 3550 1300
@@
 $EndComp
 $Comp
-L opto_board-rescue:GND-power-opto_board-rescue #PWR08
+L opto_board-rescue:GND-power-opto_board-rescue-opto_board-rescue #PWR08
 U 1 1 5E26ECD8
 P 3900 1700
@@
 pulse \ncounter 2
 $Comp
-L opto_board-rescue:R-Device R5
+L opto_board-rescue:R-Device-opto_board-rescue R5
 U 1 1 606FDE75
 P 2250 3600
@@
 Connection ~ 8500 1200
 $Comp
-L opto_board-rescue:+5V-power-board-rescue #PWR0102
+L opto_board-rescue:+5V-power-board-rescue-opto_board-rescue #PWR0102
 U 1 1 5E116347
 P 8500 950
@@
 	8200 2250 8200 2100
 $Comp
-L opto_board-rescue:GND-power-opto_board-rescue #PWR0101
+L opto_board-rescue:GND-power-opto_board-rescue-opto_board-rescue #PWR0101
 U 1 1 5E111589
 P 8200 2250
@@
 	8500 1200 9700 1200
 $Comp
-L opto_board-rescue:R-Device R2
+L opto_board-rescue:R-Device-opto_board-rescue R2
 U 1 1 5E08D481
 P 8900 1900
@@
 $EndComp
 $Comp
-L opto_board-rescue:R-Device R3
+L opto_board-rescue:R-Device-opto_board-rescue R3
 U 1 1 5E08D2BB
 P 9050 1550
@@
 Connection ~ 9300 1700
 $Comp
-L opto_board-rescue:C-Device C2
+L opto_board-rescue:C-Device-opto_board-rescue C2
 U 1 1 5E08D0D5
 P 9300 1850
@@
 	8900 1700 9300 1700
 $Comp
-L opto_board-rescue:C-Device C3
+L opto_board-rescue:C-Device-opto_board-rescue C3
 U 1 1 5E08D050
 P 9050 1350

Commit message: updated gerber files
Connections:
- net at J4.1 (Pin_1), U2.12 (PA8_Tim1ch1p): now also J4.2 (Pin_2), U1.12 (R1OUT)
- net at J5.1 (Pin_1), U2.25 (PA7_Tim1ch1n): now also J5.2 (Pin_2), U1.10 (T2IN), U1.11 (T1IN)
Changed lines of the file:
@@
 	7200 700  7000 700
 Wire Wire Line
-	4600 800  7200 800
-Wire Wire Line
-	4700 900  7200 900
+	4600 800  7100 800
+Wire Wire Line
+	4700 900  7100 900
 Wire Wire Line
 	7200 1100 6800 1100
 Wire Wire Line
-	4500 1200 7200 1200
-Wire Wire Line
-	6900 1300 7200 1300
+	4500 1200 7100 1200
+Wire Wire Line
+	6900 1300 7100 1300
 Wire Wire Line
 	4600 800  4600 2100
@@
 Wire Wire Line
 	8200 2100 9300 2100
+Wire Wire Line
+	7100 900  7100 800
+Connection ~ 7100 900
+Wire Wire Line
+	7100 900  7200 900
+Connection ~ 7100 800
+Wire Wire Line
+	7100 800  7200 800
+Wire Wire Line
+	7100 1300 7100 1200
+Connection ~ 7100 1300
+Wire Wire Line
+	7100 1300 7200 1300
+Connection ~ 7100 1200
+Wire Wire Line
+	7100 1200 7200 1200
 $EndSCHEMATC
