File: hw/kicad/opto_board.kicad_pcb (KiCad board)
At the start: 2 copper layers, 94 x 45 mm, 36 parts, among them J1 Conn_01x02, J2 DB9_Male_MountingHoles-Connec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, J4 Conn_01x03, J5 Conn_01x03, J6 Conn_01x03, J7 Conn_01x03, J8 Conn_01x03, J9 Conn_01x03, U1 MAX232N-dk_Interface-Drivers-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, U2 nucleo_nano

Commit message: improved SW/HW, added bom.txt & readme.pdf
Routing:
- net Net-(J5-Pad1): track 49.2 -> 48.4 mm
- net Net-(J4-Pad1): track 33.5 -> 32.7 mm
Other:
- board text added: "RS232 To SCPI multimeter"
- board text added: "current input"
- board text added: "fan pulse counters"
- board text added: "rs-232 opto adapter voltage"
- board text added: "temp sensors"
- board text removed: "RS232 to SCPI multimeter"
- board text removed: "Temp"
- board text removed: "current"
- board text removed: "drekkar stm32 scpi"
- board text removed: "fans"
Changed lines of the file:
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@@
     (thickness 1.6)
     (drawings 30)
-    (tracks 411)
+    (tracks 412)
     (zones 0)
     (modules 36)
@@
     (descr "Molex KK-254 Interconnect System, old/engineering part number: AE-6410-02A example for new part number: 22-27-2021, 2 Pins (http://www.molex.com/pdm_docs/sd/022272021_sd.pdf), generated with kicad-footprint-generator")
     (tags "connector Molex KK-254 side entry")
-    (fp_text reference J1 (at 5.588 -2.413 180) (layer F.SilkS)
+    (fp_text reference J1 (at 5.334 -2.921 180) (layer F.SilkS)
       (effects (font (size 1 1) (thickness 0.15)))
     )
@@
     (descr "4-lead dip package for diode bridges, row spacing 7.62 mm (300 mils), see http://cdn-reichelt.de/documents/datenblatt/A400/HDBL101G_20SERIES-TSC.pdf")
     (tags "DIL DIP PDIP 5.08mm 7.62mm 300mil")
-    (fp_text reference D7 (at 4.4196 7.7978 180) (layer F.SilkS)
+    (fp_text reference D7 (at 3.81 -3.175 180) (layer F.SilkS)
       (effects (font (size 1 1) (thickness 0.15)))
     )
@@
     (descr "Molex KK-254 Interconnect System, old/engineering part number: AE-6410-03A example for new part number: 22-27-2031, 3 Pins (http://www.molex.com/pdm_docs/sd/022272021_sd.pdf), generated with kicad-footprint-generator")
     (tags "connector Molex KK-254 side entry")
-    (fp_text reference J8 (at 2.54 4.445 180) (layer F.SilkS)
+    (fp_text reference J8 (at 5.08 4.572 180) (layer F.SilkS)
       (effects (font (size 1 1) (thickness 0.15)))
     )
@@
     (descr "C, Disc series, Radial, pin pitch=2.50mm, , diameter*width=3.8*2.6mm^2, Capacitor, http://www.vishay.com/docs/45233/krseries.pdf")
     (tags "C Disc series Radial pin pitch 2.50mm  diameter 3.8mm width 2.6mm Capacitor")
-    (fp_text reference C9 (at -1.7526 -1.3716) (layer F.SilkS)
+    (fp_text reference C9 (at -1.905 0) (layer F.SilkS)
       (effects (font (size 1 1) (thickness 0.15)))
     )
@@
     (descr "Molex KK-254 Interconnect System, old/engineering part number: AE-6410-03A example for new part number: 22-27-2031, 3 Pins (http://www.molex.com/pdm_docs/sd/022272021_sd.pdf), generated with kicad-footprint-generator")
     (tags "connector Molex KK-254 side entry")
-    (fp_text reference J9 (at 2.54 4.445 180) (layer F.SilkS)
+    (fp_text reference J9 (at -0.762 4.572 180) (layer F.SilkS)
       (effects (font (size 1 1) (thickness 0.15)))
     )
@@
     (descr "Molex KK-254 Interconnect System, old/engineering part number: AE-6410-03A example for new part number: 22-27-2031, 3 Pins (http://www.molex.com/pdm_docs/sd/022272021_sd.pdf), generated with kicad-footprint-generator")
     (tags "connector Molex KK-254 side entry")
-    (fp_text reference J7 (at 2.54 -4.12) (layer F.SilkS)
+    (fp_text reference J7 (at 7.62 -4.572) (layer F.SilkS)
       (effects (font (size 1 1) (thickness 0.15)))
     )
@@
     (descr "Molex KK-254 Interconnect System, old/engineering part number: AE-6410-03A example for new part number: 22-27-2031, 3 Pins (http://www.molex.com/pdm_docs/sd/022272021_sd.pdf), generated with kicad-footprint-generator")
     (tags "connector Molex KK-254 side entry")
-    (fp_text reference J6 (at 2.54 -4.12) (layer F.SilkS)
+    (fp_text reference J6 (at -2.54 -4.572) (layer F.SilkS)
       (effects (font (size 1 1) (thickness 0.15)))
     )
@@
       (net 5 "Net-(RX1-Pad5)"))
   )
-  (gr_text "RS232 to SCPI multimeter" (at 114.046 109.22) (layer F.SilkS)
+  (gr_text "RS232 To SCPI multimeter" (at 113.538 108.966) (layer F.SilkS)
     (effects (font (size 1 1) (thickness 0.15)))
   )
-  (gr_text fans (at 87.884 99.314) (layer F.SilkS)
+  (gr_text "fan pulse counters" (at 87.63 99.314) (layer F.SilkS)
     (effects (font (size 1 1) (thickness 0.15)))
   )
-  (gr_text current (at 84.328 67.564) (layer F.SilkS)
+  (gr_text "current input" (at 85.344 67.564) (layer F.SilkS)
     (effects (font (size 1 1) (thickness 0.15)))
   )
-  (gr_text Temp (at 115.57 67.564) (layer F.SilkS)
+  (gr_text "temp sensors" (at 115.824 67.818) (layer F.SilkS)
     (effects (font (size 1 1) (thickness 0.15)))
   )
@@
     (effects (font (size 0.8 0.8) (thickness 0.1)))
   )
-  (gr_text "drekkar stm32 scpi" (at 88.9 109.22) (layer F.SilkS)
+  (gr_text "rs-232 opto adapter voltage" (at 88.9 109.22) (layer F.SilkS)
     (effects (font (size 0.8 0.8) (thickness 0.1)))
   )
   (gr_line (start 158.75 88.9) (end 69.85 88.9) (layer F.SilkS) (width 0.2))
   (gr_line (start 114.3 109.855) (end 114.3 68.58) (layer F.SilkS) (width 0.2))
-  (gr_text "Copyright (C) 2020 \nHenrik Björkman www.eit.se/hb" (at 91.186 89.154) (layer F.SilkS)
+  (gr_text "Copyright (C) 2020 \nHenrik Björkman www.eit.se/hb" (at 90.424 89.662) (layer F.SilkS)
     (effects (font (size 0.8 0.8) (thickness 0.1)))
   )
@@
   (segment (start 83.185 85.471) (end 74.549 94.107) (width 0.5) (layer B.Cu) (net 8))
   (segment (start 74.549 97.155) (end 76.073 98.679) (width 0.5) (layer B.Cu) (net 8))
+  (segment (start 120.82 91.44) (end 121.92 91.44) (width 0.25) (layer B.Cu) (net 12))
+  (segment (start 105.025 96.52) (end 109.22 91.44) (width 0.25) (layer B.Cu) (net 12))
   (segment (start 120.084315 86.36) (end 116.633358 82.909042) (width 0.25) (layer B.Cu) (net 14))
   (segment (start 121.92 86.36) (end 120.084315 86.36) (width 0.25) (layer B.Cu) (net 14))
@@
   (segment (start 127 83.82) (end 125.476 83.82) (width 0.25) (layer F.Cu) (net 12))
   (segment (start 125.476 83.82) (end 123.952 85.344) (width 0.25) (layer F.Cu) (net 12))
-  (segment (start 109.22 91.44) (end 105.025 96.52) (width 0.25) (layer B.Cu) (net 12))
-  (segment (start 121.92 88.9) (end 118.364 88.9) (width 0.25) (layer B.Cu) (net 12))
-  (segment (start 118.364 88.9) (end 118.364 91.44) (width 0.25) (layer B.Cu) (net 12))
-  (segment (start 118.364 91.44) (end 109.22 91.44) (width 0.25) (layer B.Cu) (net 12))
-  (segment (start 121.92 91.44) (end 118.364 91.44) (width 0.25) (layer B.Cu) (net 12))
-  (segment (start 121.92 78.74) (end 124.714 78.74) (width 0.25) (layer B.Cu) (net 15))
-  (segment (start 124.714 81.28) (end 121.92 81.28) (width 0.25) (layer B.Cu) (net 15))
-  (segment (start 124.714 78.74) (end 124.714 81.28) (width 0.25) (layer B.Cu) (net 15))
-  (segment (start 125.86863 81.28) (end 124.714 81.28) (width 0.25) (layer B.Cu) (net 15))
+  (segment (start 119.126 88.9) (end 119.126 91.44) (width 0.25) (layer B.Cu) (net 12))
+  (segment (start 121.92 88.9) (end 119.126 88.9) (width 0.25) (layer B.Cu) (net 12))
+  (segment (start 119.126 91.44) (end 120.82 91.44) (width 0.25) (layer B.Cu) (net 12))
+  (segment (start 109.22 91.44) (end 119.126 91.44) (width 0.25) (layer B.Cu) (net 12))
+  (segment (start 123.952 81.28) (end 123.952 78.74) (width 0.25) (layer B.Cu) (net 15))
+  (segment (start 125.86863 81.28) (end 123.952 81.28) (width 0.25) (layer B.Cu) (net 15))
+  (segment (start 123.952 81.28) (end 121.92 81.28) (width 0.25) (layer B.Cu) (net 15))
+  (segment (start 123.952 78.74) (end 121.92 78.74) (width 0.25) (layer B.Cu) (net 15))
   (segment (start 127 86.36) (end 128.27 86.36) (width 0.25) (layer B.Cu) (net 23))
   (segment (start 128.27 86.36) (end 128.886001 85.743999) (width 0.25) (layer B.Cu) (net 23))
