File: hw/kicad/opto_board.sch (KiCad schematic (older format))
At the start: 36 parts, among them J1 Conn_01x02, J2 DB9_Male_MountingHoles-Connec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, J4 Conn_01x03, J5 Conn_01x03, J6 Conn_01x03, J7 Conn_01x03, J8 Conn_01x03, J9 Conn_01x03, U1 MAX232N-dk_Interface-Drivers-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, U2 nucleo_nano

Commit message: improved SW/HW, added bom.txt & readme.pdf
Parts:
- C1, C10, C11, C2, C3, C4, C5, C6, C7, C8, C9: symbol opto_board-rescue:C-Device-opto_board-rescue -> opto_board-rescue:C-Device
- D12, D2, D6: symbol opto_board-rescue:LED-Device-opto_board-rescue -> opto_board-rescue:LED-Device
- D4, D8: symbol opto_board-rescue:D_Zener-Device-opto_board-rescue -> opto_board-rescue:D_Zener-Device
- D7: symbol opto_board-rescue:D_Bridge_+-AA-Device-opto_board-rescue -> opto_board-rescue:D_Bridge_+-AA-Device
- J1: symbol opto_board-rescue:Conn_01x02-Connector_Generic-opto_board-rescue -> opto_board-rescue:Conn_01x02-Connector_Generic
- J4, J5, J6, J7, J8, J9: symbol opto_board-rescue:Conn_01x03-Connector_Generic-opto_board-rescue -> opto_board-rescue:Conn_01x03-Connector_Generic
- R1, R2, R3, R5, R8, R9: symbol opto_board-rescue:R-Device-opto_board-rescue -> opto_board-rescue:R-Device
- R4: value 1k -> 100; symbol opto_board-rescue:R-Device-opto_board-rescue -> opto_board-rescue:R-Device
- U2: symbol opto_board-rescue:nucleo_nano-eit_proprietary-opto_board-rescue -> opto_board-rescue:nucleo_nano-eit_proprietary
